Commit message: add assembly exaple

File: hsr_rl/models/urdf/hsrb_description/hsrb4s.urdf (robot description, URDF)
Before this commit: robot hsrb, 51 links, 50 joints
Links:
- link base_footprint: mass 13.00 -> None
- link base_link: mass 11.017971 -> 0.01
- link link_rz: mass 13.00 -> 11.017971
- link link_x: mass 13.00 -> 11.017971
- link link_y: mass 13.00 -> 11.017971
